File: SRC/ALERT_RIDER_HARDWARE/MCP73833_LIiON_BAT_CHARGER.kicad_sch (KiCad schematic)
At the start: 14 parts, among them U7 MCP73833-AMI_UN

Commit message: complete Pa8-Pa7 LED placement maximized all files generated
Parts:
- D2, D5: footprint LED_SMD:LED_0603_1608Metric -> LED_SMD:LED_0402_1005Metric
Changed lines of the file:
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@@
       (effects (font (size 1.27 1.27)) (justify right))
     )
-    (property "Footprint" "LED_SMD:LED_0603_1608Metric" (at 201.93 92.075 0)
+    (property "Footprint" "LED_SMD:LED_0402_1005Metric" (at 201.93 92.075 0)
       (effects (font (size 1.27 1.27)) hide)
     )
@@
       (effects (font (size 1.27 1.27)) (justify right))
     )
-    (property "Footprint" "LED_SMD:LED_0603_1608Metric" (at 190.5 92.075 0)
+    (property "Footprint" "LED_SMD:LED_0402_1005Metric" (at 190.5 92.075 0)
       (effects (font (size 1.27 1.27)) hide)
     )

Commit message: alert rider updated complete internal rc HSI version
Connections:
- net +3V3 is gone; now on net +5V: R15.1, R47.1
Changed lines of the file:
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@@
 (kicad_sch (version 20230121) (generator eeschema)
   (paper "A4")
+  (junction (at 196.85 73.66) (diameter 0) (color 0 0 0 0)
+  )
   (junction (at 110.49 105.41) (diameter 0) (color 0 0 0 0)
   )
@@
   (junction (at 177.165 107.95) (diameter 0) (color 0 0 0 0)
   )
+  (wire (pts (xy 190.5 73.66) (xy 196.85 73.66))
+    (stroke (width 0) (type default))
+  )
   (wire (pts (xy 130.81 117.475) (xy 130.81 118.745))
     (stroke (width 0) (type default))
@@
     (stroke (width 0) (type default))
   )
-  (wire (pts (xy 201.93 74.295) (xy 201.93 77.47))
+  (wire (pts (xy 201.93 73.66) (xy 201.93 77.47))
     (stroke (width 0) (type default))
   )
@@
     (stroke (width 0) (type default))
   )
+  (wire (pts (xy 196.85 73.66) (xy 201.93 73.66))
+    (stroke (width 0) (type default))
+  )
   (wire (pts (xy 130.81 105.41) (xy 110.49 105.41))
     (stroke (width 0) (type default))
@@
     (stroke (width 0) (type default))
   )
-  (wire (pts (xy 190.5 74.295) (xy 190.5 77.47))
+  (wire (pts (xy 190.5 73.66) (xy 190.5 77.47))
     (stroke (width 0) (type default))
   )
@@
     )
   )
-  (symbol (lib_id "power:+3V3") (at 201.93 74.295 0) (unit 1)
-    (in_bom yes) (on_board yes) (dnp no) (fields_autoplaced)
-    (property "Reference" "#PWR061" (at 201.93 78.105 0)
-      (effects (font (size 1.27 1.27)) hide)
-    )
-    (property "Value" "+3V3" (at 201.93 71.12 0)
-      (effects (font (size 1.27 1.27)))
-    )
-    (property "Footprint" "" (at 201.93 74.295 0)
-      (effects (font (size 1.27 1.27)) hide)
-    )
-    (property "Datasheet" "" (at 201.93 74.295 0)
-      (effects (font (size 1.27 1.27)) hide)
-    )
-    (pin "1")
-    (instances
-      (project "ALERT_RIDER_HARDWARE"
-        (path "/6bd12930-91c7-432a-9f98-f9ae5061d3a7/dc7ea31c-f73c-4b6f-84ef-6d55208cc8ab"
-          (reference "#PWR061") (unit 1)
-        )
-      )
-    )
-  )
   (symbol (lib_id "power:+5V") (at 167.005 83.185 0) (mirror y) (unit 1)
     (in_bom yes) (on_board yes) (dnp no) (fields_autoplaced)
@@
     )
   )
-  (symbol (lib_id "power:+3V3") (at 190.5 74.295 0) (unit 1)
-    (in_bom yes) (on_board yes) (dnp no) (fields_autoplaced)
-    (property "Reference" "#PWR028" (at 190.5 78.105 0)
-      (effects (font (size 1.27 1.27)) hide)
-    )
-    (property "Value" "+3V3" (at 190.5 71.12 0)
-      (effects (font (size 1.27 1.27)))
-    )
-    (property "Footprint" "" (at 190.5 74.295 0)
-      (effects (font (size 1.27 1.27)) hide)
-    )
-    (property "Datasheet" "" (at 190.5 74.295 0)
-      (effects (font (size 1.27 1.27)) hide)
-    )
-    (pin "1")
-    (instances
-      (project "ALERT_RIDER_HARDWARE"
-        (path "/6bd12930-91c7-432a-9f98-f9ae5061d3a7/dc7ea31c-f73c-4b6f-84ef-6d55208cc8ab"
-          (reference "#PWR028") (unit 1)
-        )
-      )
-    )
-  )
   (symbol (lib_id "power:GND") (at 158.75 116.205 0) (mirror y) (unit 1)
     (in_bom yes) (on_board yes) (dnp no) (fields_autoplaced)
@@
         )
       )
+    )
+  )
+  (symbol (lib_id "power:+5V") (at 196.85 73.66 0) (mirror y) (unit 1)
+    (in_bom yes) (on_board yes) (dnp no) (fields_autoplaced)
+    (property "Reference" "#PWR017" (at 196.85 77.47 0)
+      (effects (font (size 1.27 1.27)) hide)
+    )
+    (property "Value" "+5V" (at 196.85 68.58 0)
+      (effects (font (size 1.27 1.27)))
+    )
+    (property "Footprint" "" (at 196.85 73.66 0)
+      (effects (font (size 1.27 1.27)) hide)
+    )
+    (property "Datasheet" "" (at 196.85 73.66 0)
+      (effects (font (size 1.27 1.27)) hide)
+    )
+    (pin "1")
+    (instances
+      (project "ALERT_RIDER_HARDWARE"
+        (path "/6bd12930-91c7-432a-9f98-f9ae5061d3a7/dc7ea31c-f73c-4b6f-84ef-6d55208cc8ab"
+          (reference "#PWR017") (unit 1)
+        )
+      )
